File: zudo-bus.kicad_sch (KiCad schematic)
At the start: 56 parts, among them P1 WJ500V-5.08-2P-14-00A, P2 WJ500V-5.08-2P-14-00A, U10 2541WR-2X08P, U11 2541WR-2X08P, U12 1217754-1, U13 1217754-1, U14 1217754-1, U15 1217754-1, U2 2541WR-2X08P, U3 YLED0603YG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

Commit message: initialized sch
Parts:
- removed C1, C10, C11, C12, C13, C14, C15, C16, C2, C20, C23, C3, C4, C5, C6, C7, C8, C9: CC0603KRX7R9BB104, easyeda2kicad:C0603, symbol zudo-bus:CC0603KRX7R9BB104
- removed C17, C18, C19, C22: CL21A226MAQNNNE, zudo-bus:C0805, symbol zudo-bus-new-protection:CL21A226MAQNNNE
- removed C21: CL21A106KAYNNNE, samsung-caps:C0805, symbol samsung-caps:CL21A106KAYNNNE
- removed D1, D3: SMF12CA_C353317, zudo-bus:SOD-123FL_L2.8-W1.8-LS3.7-BI, symbol zudo-bus-new-protection:SMF12CA_C353317
- removed D2: SMF5.0CA_C908214, :SOD-123_L2.8-W1.8-LS3.7-BI, symbol zudo-bus-protection:SMF5.0CA_C908214
- removed D4, D5: SS14, zudo-bus:SMA_L4.2-W2.6-LS5.0-RD_1, symbol zudo-bus-new-protection:SS14
- removed D6, D7, D8, D9: SM4007PL, easyeda2kicad:SOD-123F_L2.8-W1.8-LS3.7-RD, symbol zudo-bus:SM4007PL
- removed F1, F2: BSMD1812-200-30V, :F1812, symbol zudo-bus-protection:BSMD1812-200-30V
- removed F3, F4: BSMD1812-150-33V, :F1812, symbol zudo-bus-protection:BSMD1812-150-33V
- removed H1: Header-Male-2.54_1x3, easyeda2kicad:HDR-TH_3P-P2.54-V-M-1, symbol zudo-bus:Header-Male-2.54_1x3
- removed LED1: KT-0603R, easyeda2kicad:LED0603-RD, symbol zudo-bus:KT-0603R
- removed P1, P2: WJ500V-5.08-2P-14-00A, easyeda2kicad:CONN-TH_2P-P5.00_WJ500V-5.08-2P, symbol zudo-bus:WJ500V-5.08-2P-14-00A
- removed R1: 0805W8J0102T5E, easyeda2kicad:R0805, symbol zudo-bus:0805W8J0102T5E
- removed TP1: TestPoint, symbol Connector:TestPoint
- removed U10, U11, U2, U5, U6, U7, U8, U9: 2541WR-2X08P, easyeda2kicad:HDR-TH_16P-P2.54-H-M-R2-C8-S2.54, symbol zudo-bus:2541WR-2X08P
- removed U12, U13, U14, U15: 1217754-1, easyeda2kicad:CONN-TH_1217754-1, symbol zudo-bus:1217754-1
- removed U3: YLED0603YG, easyeda2kicad:LED0603-FD, symbol zudo-bus:YLED0603YG
- removed U4: NCD1608A1, easyeda2kicad:LED0603-RD, symbol zudo-bus:NCD1608A1
