File: rail.kicad_sch (KiCad schematic)
At the start: 24 parts, among them J101 2541WR-2X08P, J102 2541WR-2X08P, J103 2541WR-2X08P, J104 2541WR-2X08P, J105 2541WR-2X08P, J106 2541WR-2X08P, J107 2541WR-2X08P, J108 2541WR-2X08P

Commit message: Update KiCad schematic and PCB layout
- Adjust IDC header positions and rotations in rail schematic
- Update PCB layout with component placements
- Update project configuration
Connections:
- net +12V rail: now also J101.7, J101.8, J102.7, J102.8, J103.7, J103.8, J104.7, J104.8, J105.7, J105.8, J106.7, J106.8, J107.7, J107.8, J108.7, J108.8; no longer J101.10, J101.9, J102.10, J102.9, J103.10, J103.9, J104.10, J104.9, J105.10, J105.9, J106.10, J106.9, J107.10, J107.9, J108.10, J108.9
- net +5V rail: now also J101.5, J101.6, J102.5, J102.6, J103.5, J103.6, J104.5, J104.6, J105.5, J105.6, J106.5, J106.6, J107.5, J107.6, J108.5, J108.6; no longer J101.11, J101.12, J102.11, J102.12, J103.11, J103.12, J104.11, J104.12, J105.11, J105.12, J106.11, J106.12, J107.11, J107.12, J108.11, J108.12
- net -12V rail: now also J101.15, J101.16, J102.15, J102.16, J103.15, J103.16, J104.15, J104.16, J105.15, J105.16, J106.15, J106.16, J107.15, J107.16, J108.15, J108.16; no longer J101.1, J101.2, J102.1, J102.2, J103.1, J103.2, J104.1, J104.2, J105.1, J105.2, J106.1, J106.2, J107.1, J107.2, J108.1, J108.2
- net CV rail: now also J101.3, J101.4, J102.3, J102.4, J103.3, J103.4, J104.3, J104.4, J105.3, J105.4, J106.3, J106.4, J107.3, J107.4, J108.3, J108.4; no longer J101.13, J101.14, J102.13, J102.14, J103.13, J103.14, J104.13, J104.14, J105.13, J105.14, J106.13, J106.14, J107.13, J107.14, J108.13, J108.14
- net GATE rail: now also J101.1, J101.2, J102.1, J102.2, J103.1, J103.2, J104.1, J104.2, J105.1, J105.2, J106.1, J106.2, J107.1, J107.2, J108.1, J108.2; no longer J101.15, J101.16, J102.15, J102.16, J103.15, J103.16, J104.15, J104.16, J105.15, J105.16, J106.15, J106.16, J107.15, J107.16, J108.15, J108.16
- net GND: now also J101.10, J101.11, J101.12, J101.13, J101.14, J101.9, J102.10, J102.11, J102.12, J102.13, J102.14, J102.9, J103.10, J103.11, J103.12, J103.13, J103.14, J103.9, J104.10, J104.11, J104.12, J104.13, J104.14, J104.9, J105.10, J105.11, J105.12, J105.13, J105.14, J105.9, J106.10, J106.11, J106.12, J106.13, J106.14, J106.9, J107.10, J107.11, J107.12, J107.13, J107.14, J107.9, J108.10, J108.11, J108.12, J108.13, J108.14, J108.9; no longer J101.3, J101.4, J101.5, J101.6, J101.7, J101.8, J102.3, J102.4, J102.5, J102.6, J102.7, J102.8, J103.3, J103.4, J103.5, J103.6, J103.7, J103.8, J104.3, J104.4, J104.5, J104.6, J104.7, J104.8, J105.3, J105.4, J105.5, J105.6, J105.7, J105.8, J106.3, J106.4, J106.5, J106.6, J106.7, J106.8, J107.3, J107.4, J107.5, J107.6, J107.7, J107.8, J108.3, J108.4, J108.5, J108.6, J108.7, J108.8
Other:
- moved on the sheet: J101, J102, J103, J104, J105, J106, J107, J108
Changed lines of the file:
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@@
 	(symbol
 		(lib_id "zudo-bus:2541WR-2X08P")
-		(at 179.07 92.71 0)
+		(at 179.07 92.71 180)
 		(unit 1)
 		(exclude_from_sim no)
@@
 		)
 		(property "Value" "2541WR-2X08P"
-			(at 179.07 78.74 0)
+			(at 179.07 106.68 0)
 			(effects
 				(font
@@
 		)
 		(property "Footprint" "easyeda2kicad:HDR-TH_16P-P2.54-H-M-R2-C8-S2.54"
-			(at 179.07 109.22 0)
+			(at 179.07 76.2 0)
 			(effects
 				(font
@@
 		)
 		(property "LCSC Part" "C5383092"
-			(at 179.07 111.76 0)
+			(at 179.07 73.66 0)
 			(effects
 				(font
@@
 	(symbol
 		(lib_id "zudo-bus:2541WR-2X08P")
-		(at 100.33 43.18 0)
+		(at 100.33 43.18 180)
 		(unit 1)
 		(exclude_from_sim no)
@@
 		)
 		(property "Value" "2541WR-2X08P"
-			(at 100.33 29.21 0)
+			(at 100.33 57.15 0)
 			(effects
 				(font
@@
 		)
 		(property "Footprint" "easyeda2kicad:HDR-TH_16P-P2.54-H-M-R2-C8-S2.54"
-			(at 100.33 59.69 0)
+			(at 100.33 26.67 0)
 			(effects
 				(font
@@
 		)
 		(property "LCSC Part" "C5383092"
-			(at 100.33 62.23 0)
+			(at 100.33 24.13 0)
 			(effects
 				(font
@@
 	(symbol
 		(lib_id "zudo-bus:2541WR-2X08P")
-		(at 100.33 92.71 0)
+		(at 100.33 92.71 180)
 		(unit 1)
 		(exclude_from_sim no)
@@
 		)
 		(property "Value" "2541WR-2X08P"
-			(at 100.33 78.74 0)
+			(at 100.33 106.68 0)
 			(effects
 				(font
@@
 		)
 		(property "Footprint" "easyeda2kicad:HDR-TH_16P-P2.54-H-M-R2-C8-S2.54"
-			(at 100.33 109.22 0)
+			(at 100.33 76.2 0)
 			(effects
 				(font
@@
 		)
 		(property "LCSC Part" "C5383092"
-			(at 100.33 111.76 0)
+			(at 100.33 73.66 0)
 			(effects
 				(font
@@
 	(symbol
 		(lib_id "zudo-bus:2541WR-2X08P")
-		(at 179.07 140.97 0)
+		(at 179.07 140.97 180)
 		(unit 1)
 		(exclude_from_sim no)
@@
 		)
 		(property "Value" "2541WR-2X08P"
-			(at 179.07 127 0)
+			(at 179.07 154.94 0)
 			(effects
 				(font
@@
 		)
 		(property "Footprint" "easyeda2kicad:HDR-TH_16P-P2.54-H-M-R2-C8-S2.54"
-			(at 179.07 157.48 0)
+			(at 179.07 124.46 0)
 			(effects
 				(font
@@
 		)
 		(property "LCSC Part" "C5383092"
-			(at 179.07 160.02 0)
+			(at 179.07 121.92 0)
 			(effects
 				(font
@@
 	(symbol
 		(lib_id "zudo-bus:2541WR-2X08P")
-		(at 252.73 92.71 0)
+		(at 252.73 92.71 180)
 		(unit 1)
 		(exclude_from_sim no)
@@
 		)
 		(property "Value" "2541WR-2X08P"
-			(at 252.73 78.74 0)
+			(at 252.73 106.68 0)
 			(effects
 				(font
@@
 		)
 		(property "Footprint" "easyeda2kicad:HDR-TH_16P-P2.54-H-M-R2-C8-S2.54"
-			(at 252.73 109.22 0)
+			(at 252.73 76.2 0)
 			(effects
 				(font
@@
 		)
 		(property "LCSC Part" "C5383092"
-			(at 252.73 111.76 0)
+			(at 252.73 73.66 0)
 			(effects
 				(font
@@
 	(symbol
 		(lib_id "zudo-bus:2541WR-2X08P")
-		(at 252.73 43.18 0)
+		(at 252.73 43.18 180)
 		(unit 1)
 		(exclude_from_sim no)
@@
 		)
 		(property "Value" "2541WR-2X08P"
-			(at 252.73 29.21 0)
+			(at 252.73 57.15 0)
 			(effects
 				(font
@@
 		)
 		(property "Footprint" "easyeda2kicad:HDR-TH_16P-P2.54-H-M-R2-C8-S2.54"
-			(at 252.73 59.69 0)
+			(at 252.73 26.67 0)
 			(effects
 				(font
@@
 		)
 		(property "LCSC Part" "C5383092"
-			(at 252.73 62.23 0)
+			(at 252.73 24.13 0)
 			(effects
 				(font
@@
 	(symbol
 		(lib_id "zudo-bus:2541WR-2X08P")
-		(at 100.33 140.97 0)
+		(at 100.33 140.97 180)
 		(unit 1)
 		(exclude_from_sim no)
@@
 		)
 		(property "Value" "2541WR-2X08P"
-			(at 100.33 127 0)
+			(at 100.33 154.94 0)
 			(effects
 				(font
@@
 		)
 		(property "Footprint" "easyeda2kicad:HDR-TH_16P-P2.54-H-M-R2-C8-S2.54"
-			(at 100.33 157.48 0)
+			(at 100.33 124.46 0)
 			(effects
 				(font
@@
 		)
 		(property "LCSC Part" "C5383092"
-			(at 100.33 160.02 0)
+			(at 100.33 121.92 0)
 			(effects
 				(font
@@
 	(symbol
 		(lib_id "zudo-bus:2541WR-2X08P")
-		(at 179.07 43.18 0)
+		(at 179.07 43.18 180)
 		(unit 1)
 		(exclude_from_sim no)
@@
 		)
 		(property "Value" "2541WR-2X08P"
-			(at 179.07 29.21 0)
+			(at 179.07 57.15 0)
 			(effects
 				(font
@@
 		)
 		(property "Footprint" "easyeda2kicad:HDR-TH_16P-P2.54-H-M-R2-C8-S2.54"
-			(at 179.07 59.69 0)
+			(at 179.07 26.67 0)
 			(effects
 				(font
@@
 		)
 		(property "LCSC Part" "C5383092"
-			(at 179.07 62.23 0)
-			(effects
-				(font
+			(at 179.07 24.13 0)
+			(effects
+				(font
