File: zudo-bus.kicad_pcb (KiCad board)
At the start: 2 copper layers, 205 x 39 mm, 65 parts, among them J101 2541WR-2X08P, J102 2541WR-2X08P, J103 2541WR-2X08P, J104 2541WR-2X08P, J105 2541WR-2X08P, J106 2541WR-2X08P, J107 2541WR-2X08P, J108 2541WR-2X08P, P1 WJ500V-5.08-2P-14-00A, P2 WJ500V-5.08-2P-14-00A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

Commit message: Add custom footprints and update PCB layout
- Add eurorack-power-16pin footprint with custom silkscreen
- Add power-faston-pin footprint for FASTON connectors
- Update PCB layout with component placements
- Add design resource file (zudo-bus-svg.ai)
Parts:
- added REF**: MountingHole_3.2mm_M3, MountingHole:MountingHole_3.2mm_M3, F.Cu at (100.5, 26.5)
- added REF**: MountingHole_3.2mm_M3, MountingHole:MountingHole_3.2mm_M3, F.Cu at (64.5, 12.5)
- added REF**: MountingHole_3.2mm_M3, MountingHole:MountingHole_3.2mm_M3, F.Cu at (136.5, 12.5)
- J101, J102, J103, J104, J105, J106, J107, J108: footprint easyeda2kicad:HDR-TH_16P-P2.54-H-M-R2-C8-S2.54 -> zudo-bus:eurorack-power-16pin
- P3, P4, P5, P6: footprint easyeda2kicad:CONN-TH_1217754-1 -> zudo-bus:power-faston-pin
Routing:
- net CV rail: vias 8 -> 7
Other:
- board size 205 x 39 mm -> 203 x 39 mm
- board text added: "+5V | +12V | GND | -12V"
